Commit message: Update robot4.xacro

File: robot_urdf-ros2/urdf/robot4.xacro (robot description, xacro)
@@ -2,4 +2,5 @@
 <robot xmlns:xacro="http://www.ros.org/wiki/xacro" name="robot4_xacro">
 <xacro:include filename="$(find robot_urdf)/urdf/robot4.gazebo"/>
+<xacro:include filename="$(find robot_urdf)/urdf/materials.xacro" />
 	<xacro:property name="length_wheel" value="0.04" />
 	<xacro:property name="radius_wheel" value="0.1" />
@@ -11,163 +12,139 @@
                </inertial>
 	</xacro:macro>
-    <xacro:macro name="wheel_geometry">
+    	<xacro:macro name="wheel_geometry">
 		<geometry>
-       			<cylinder length="${length_wheel}" radius="${radius_wheel}"/>
-     	</geometry>
+			<cylinder length="${length_wheel}" radius="${radius_wheel}"/>
+     		</geometry>
 	</xacro:macro>
-  <material name="black">
-    <color rgba="0.0 0.0 0.0 1.0"/>
-  </material>
-  <material name="blue">
-    <color rgba="0.203125 0.23828125 0.28515625 1.0"/>
-  </material>
-  <material name="green">
-    <color rgba="0.0 0.8 0.0 1.0"/>
-  </material>
-  <material name="grey">
-    <color rgba="0.2 0.2 0.2 1.0"/>
-  </material>
-  <material name="orange">
-    <color rgba="1.0 0.423529411765 0.0392156862745 1.0"/>
-  </material>
-  <material name="brown">
-    <color rgba="0.870588235294 0.811764705882 0.764705882353 1.0"/>
-  </material>
-  <material name="red">
-    <color rgba="0.80078125 0.12890625 0.1328125 1.0"/>
-  </material>
-  <material name="white">
-    <color rgba="1.0 1.0 1.0 1.0"/>
-  </material>
-	  <link name="link_chassis">
-    <!-- pose and inertial -->
-    <pose>0 0 0.1 0 0 0</pose>
-    <inertial>
-      <mass value="5"/>
-      <origin rpy="0 0 0" xyz="0 0 0.1"/>
-      <inertia ixx="0.0395416666667" ixy="0" ixz="0" iyy="0.106208333333" iyz="0" izz="0.106208333333"/>
-    </inertial>
-    <!-- body -->
-    <collision name="collision_chassis">
-      <geometry>
-        <box size="0.5 0.3 0.07"/>
-      </geometry>
-    </collision>
-    <visual>
-      <origin rpy="0 0 0" xyz="0 0 0"/>
-      <geometry>
-        <box size="0.5 0.3 0.07"/>
-      </geometry>
-      <material name="blue"/>
-    </visual>
-    <!-- caster front -->
-    <collision name="caster_front_collision">
-      <origin rpy=" 0 0 0" xyz="0.35 0 -0.05"/>
-      <geometry>
-        <sphere radius="0.05"/>
-      </geometry>
-    </collision>
-    <visual name="caster_front_visual">
-      <origin rpy=" 0 0 0" xyz="0.2 0 -0.05"/>
-      <geometry>
-        <sphere radius="0.05"/>
-      </geometry>
-    </visual>
-  </link>
-   <link name="link_right_wheel">
-    <xacro:default_inertial mass="0.2"/>
-    <collision name="link_right_wheel_collision">
-      <origin rpy="0 1.5707 1.5707" xyz="0 0 0"/>
-      <xacro:wheel_geometry />
-    </collision>
-    <visual name="link_right_wheel_visual">
-      <origin rpy="0 1.5707 1.5707" xyz="0 0 0"/>
-      <xacro:wheel_geometry />
-      <material name="red"/>
-    </visual>
-  </link>
-   <link name="link_left_wheel">
-    <xacro:default_inertial mass="0.2"/>
-    <collision name="link_left_wheel_collision">
-      <origin rpy="0 1.5707 1.5707" xyz="0 0 0"/>
-      <xacro:wheel_geometry />
-    </collision>
-    <visual name="link_left_wheel_visual">
-      <origin rpy="0 1.5707 1.5707" xyz="0 0 0"/>
-      <xacro:wheel_geometry />
-      <material name="red"/>
-    </visual>
-  </link>
-  <joint name="joint_right_wheel" type="continuous">
-    <origin rpy="0 0 0" xyz="-0.05 0.15 0"/>
-    <child link="link_right_wheel"/>
-    <parent link="link_chassis"/>
-    <axis rpy="0 0 0" xyz="0 1 0"/>
-    <limit effort="10000" velocity="1000"/>
-    <joint_properties damping="1.0" friction="1.0"/>
-  </joint>
-  <joint name="joint_left_wheel" type="continuous">
-    <origin rpy="0 0 0" xyz="-0.05 -0.15 0"/>
-    <child link="link_left_wheel"/>
-    <parent link="link_chassis"/>
-    <axis rpy="0 0 0" xyz="0 1 0"/>
-    <limit effort="10000" velocity="1000"/>
-    <joint_properties damping="1.0" friction="1.0"/>
-  </joint>
-  <link name="link_camera_rot">
-    <collision>
-      <origin xyz="0 0 0.05" rpy="0 0 0"/>
-      <geometry>
-	<box size="0.06 0.06 0.1"/>
-      </geometry>
-    </collision>
-	  <visual>
-    <origin rpy="0 0 0.05" xyz="0 0 0"/>
-    <geometry>
-	<box size="0.06 0.06 0.1"/>
-    </geometry>
-    <material name="white"/>
-  </visual>
-  <inertial>
-      <mass value="0.1" />
-      <origin xyz="0 0 0" rpy="0 0 0"/>
-      <inertia ixx="1e-4" ixy="0" ixz="0" iyy="1e-4" iyz="0" izz="4e-5" />
-   </inertial>
-  </link>
-  <link name="camera_link">
-	    <collision>
-	      <origin xyz="0 0 0.075" rpy="0 0 0"/>
-	      <geometry>
-		<box size="0.05 0.05 0.05"/>
-	      </geometry>
-	    </collision>
-	    <visual>
-	      <origin xyz="0 0 0.075" rpy="0 0 0"/>
-	      <geometry>
-		<box size="0.05 0.05 0.05"/>
-	      </geometry>
-	      <material name="red">
+<link name="link_chassis">
+	<!-- pose and inertial -->
+		<pose>0 0 0.1 0 0 0</pose>
+		<inertial>
+			<mass value="5"/>
+			<origin rpy="0 0 0" xyz="0 0 0.1"/>
+			<inertia ixx="0.0395416666667" ixy="0" ixz="0" iyy="0.106208333333" iyz="0" izz="0.106208333333"/>
+		</inertial>
+	<!-- body -->
+		<collision name="collision_chassis">
+			<geometry>
+				<box size="0.5 0.3 0.07"/>
+			</geometry>
+		</collision>
+		<visual>
+			<origin rpy="0 0 0" xyz="0 0 0"/>
+			<geometry>
+				<box size="0.5 0.3 0.07"/>
+			</geometry>
+			<material name="blue"/>
+		</visual>
+	<!-- caster front -->
+		<collision name="caster_front_collision">
+		<origin rpy=" 0 0 0" xyz="0.35 0 -0.05"/>
+		<geometry>
+			<sphere radius="0.05"/>
+		</geometry>
+		</collision>
+		<visual name="caster_front_visual">
+		<origin rpy=" 0 0 0" xyz="0.2 0 -0.05"/>
+		<geometry>
+			<sphere radius="0.05"/>
+		</geometry>
+		</visual>
+</link>
+<link name="link_right_wheel">
+	<xacro:default_inertial mass="0.2"/>
+	<collision name="link_right_wheel_collision">
+	  <origin rpy="0 1.5707 1.5707" xyz="0 0 0"/>
+	  <xacro:wheel_geometry />
+	</collision>
+	<visual name="link_right_wheel_visual">
+	  <origin rpy="0 1.5707 1.5707" xyz="0 0 0"/>
+	  <xacro:wheel_geometry />
+	  <material name="red"/>
+	</visual>
+</link>
+<link name="link_left_wheel">
+	<xacro:default_inertial mass="0.2"/>
+	<collision name="link_left_wheel_collision">
+	  <origin rpy="0 1.5707 1.5707" xyz="0 0 0"/>
+	  <xacro:wheel_geometry />
+	</collision>
+	<visual name="link_left_wheel_visual">
+	  <origin rpy="0 1.5707 1.5707" xyz="0 0 0"/>
+	  <xacro:wheel_geometry />
+	  <material name="red"/>
+	</visual>
+</link>
+<joint name="joint_right_wheel" type="continuous">
+	<origin rpy="0 0 0" xyz="-0.05 0.15 0"/>
+	<child link="link_right_wheel"/>
+	<parent link="link_chassis"/>
+	<axis rpy="0 0 0" xyz="0 1 0"/>
+	<limit effort="10000" velocity="1000"/>
+	<joint_properties damping="1.0" friction="1.0"/>
+</joint>
+<joint name="joint_left_wheel" type="continuous">
+	<origin rpy="0 0 0" xyz="-0.05 -0.15 0"/>
+	<child link="link_left_wheel"/>
+	<parent link="link_chassis"/>
+	<axis rpy="0 0 0" xyz="0 1 0"/>
+	<limit effort="10000" velocity="1000"/>
+	<joint_properties damping="1.0" friction="1.0"/>
+</joint>
+<link name="link_camera_rot">
+	<collision>
+		<origin xyz="0 0 0.05" rpy="0 0 0"/>
+		<geometry>
+			<box size="0.06 0.06 0.1"/>
+		</geometry>
+	</collision>
+	<visual>
+		<origin rpy="0 0 0.05" xyz="0 0 0"/>
+		<geometry>
+			<box size="0.06 0.06 0.1"/>
+		</geometry>
+		<material name="white"/>
+	</visual>
+	<inertial>
+		<mass value="0.1" />
+		<origin xyz="0 0 0" rpy="0 0 0"/>
+		<inertia ixx="1e-4" ixy="0" ixz="0" iyy="1e-4" iyz="0" izz="4e-5" />
+	</inertial>
+</link>
+<link name="camera_link">
+	<collision>
+		<origin xyz="0 0 0.075" rpy="0 0 0"/>
+		<geometry>
+			<box size="0.05 0.05 0.05"/>
+		</geometry>
+	</collision>
+	<visual>
+		<origin xyz="0 0 0.075" rpy="0 0 0"/>
+		<geometry>
+			<box size="0.05 0.05 0.05"/>
+		</geometry>
+		<material name="red">
 		<color rgba="1 0 0 1"/>
-	      </material>
-	    </visual>
-	    <inertial>
-	      <mass value="1e-5" />
-	      <origin xyz="0 0 0" rpy="0 0 0"/>
-	      <inertia ixx="1e-6" ixy="0" ixz="0" iyy="1e-6" iyz="0" izz="1e-6" />
-	    </inertial>
-  </link>
-   <joint name="joint_camera_rot" type="continuous">
-    <origin rpy="0 0 0" xyz="0.1 0 0.085"/>
-    <child link="link_camera_rot"/>
-    <parent link="link_chassis"/>
-    <axis rpy="0 0 0" xyz="0 0 1"/>
-    <limit effort="10000" velocity="1000"/>
-    <joint_properties damping="1.0" friction="1.0"/>
-  </joint>
-  <joint name="camera_joint" type="fixed">
-	    <axis xyz="0 1 0" />
-	    <origin xyz="0 0 0" rpy="0 0 0"/>
-	    <parent link="link_camera_rot"/>
-	    <child link="camera_link"/>
-	 </joint>
+		</material>
+	</visual>
+	<inertial>
+		<mass value="1e-5" />
+		<origin xyz="0 0 0" rpy="0 0 0"/>
+		<inertia ixx="1e-6" ixy="0" ixz="0" iyy="1e-6" iyz="0" izz="1e-6" />
+	</inertial>
+</link>
+<joint name="joint_camera_rot" type="continuous">
+	<origin rpy="0 0 0" xyz="0.1 0 0.085"/>
+	<child link="link_camera_rot"/>
+	<parent link="link_chassis"/>
+	<axis rpy="0 0 0" xyz="0 0 1"/>
+	<limit effort="10000" velocity="1000"/>
+	<joint_properties damping="1.0" friction="1.0"/>
+</joint>
+<joint name="camera_joint" type="fixed">
+	<axis xyz="0 1 0" />
+	<origin xyz="0 0 0" rpy="0 0 0"/>
+	<parent link="link_camera_rot"/>
+	<child link="camera_link"/>
+</joint>
 </robot>

Commit message: Update robot4.xacro

File: robot_urdf-ros2/urdf/robot4.xacro (robot description, xacro)
@@ -31,5 +31,5 @@
 		<origin rpy="0 0 0" xyz="${origin_xyz}"/>
 		<child link="${child}"/>
-		<parent link="base_link"/>
+		<parent link="link_chassis"/>
 		<axis rpy="0 0 0" xyz="0 1 0"/>
 		<limit effort="10000" velocity="1000"/>
@@ -37,5 +37,5 @@
 	</joint>
 </xacro:macro>
-<link name="base_link">
+<link name="link_chassis">
 	<!-- pose and inertial -->
 	<pose>0 0 0.1 0 0 0</pose>
@@ -93,7 +93,7 @@
   	</inertial>
 	<collision>
-  	  <origin xyz="0 0 0.05" rpy="0 0 0"/>
+  	  <origin xyz="0 0 0" rpy="0 0 0"/>
       <geometry>
-        <cylinder radius="0.05" length="0.08"/>
+        <cylinder radius="0.05" length="0.1"/>
       </geometry>
   	</collision>
@@ -101,5 +101,5 @@
   	  <origin xyz="0 0 0" rpy="0 0 0"/>
       <geometry>
-        <cylinder radius="0.05" length="0.08"/>
+        <cylinder radius="0.05" length="0.1"/>
       </geometry>
       <material name="red" />
@@ -136,5 +136,5 @@
 </link>
 <joint name="camera_joint" type="fixed">
-	<axis xyz="0 1 0" />
+	<axis xyz="0 0 1" />
 	<origin xyz="0 0 0" rpy="0 0 0"/>
 	<parent link="link_camera_rot"/>

Commit message: Update robot4.xacro

File: robot_urdf-ros2/urdf/robot4.xacro (robot description, xacro)
@@ -113,5 +113,5 @@
 	<limit effort="1.0" lower="-3.14" upper="3.14" velocity="10.0"/>
 </joint>
-<link name="camera">
+<link name="camera_link">
 	<collision>
 		<origin xyz="0 0 0.075" rpy="0 0 0"/>
@@ -139,5 +139,5 @@
 	<origin xyz="0 0 0" rpy="0 0 0"/>
 	<parent link="link_camera_rot"/>
-	<child link="camera"/>
+	<child link="camera_link"/>
 </joint>
 </robot>

Commit message: Update robot4.xacro
Asse camera rotazione da 0 rad a 6.29 rad (2pi)

File: robot_urdf-ros2/urdf/robot4.xacro (robot description, xacro)
@@ -111,5 +111,5 @@
 	<parent link="link_chassis"/>
 	<axis rpy="0 0 0" xyz="0 0 1"/>
-	<limit effort="1.0" lower="-3.14" upper="3.14" velocity="10.0"/>
+	<limit effort="1.0" lower="0" upper="6.29" velocity="10.0"/>
 </joint>
 <link name="camera_link">

Commit message: XACRO
mosso il sistema di riferimento sopra, così si vede effettivamnete da li

In ACTION sto aggiungendo le matrici per la relazione tra camera e sitsema di riferimento del robot

File: robot_urdf-ros2/urdf/robot4.xacro (robot description, xacro)
@@ -121,5 +121,5 @@
 	</collision>
 	<visual>
-		<origin xyz="0 0 0.075" rpy="0 0 0"/>
+		<origin xyz="0 0 0" rpy="0 0 0"/>
 		<geometry>
 			<box size="0.05 0.05 0.05"/>
@@ -137,5 +137,5 @@
 <joint name="camera_joint" type="fixed">
 	<axis xyz="0 0 1" />
-	<origin xyz="0 0 0" rpy="0 0 0"/>
+	<origin xyz="0 0 0.075" rpy="0 0 0"/>
 	<parent link="link_camera_rot"/>
 	<child link="camera_link"/>
